Commit message: fix v1 urdf, hip's axis

File: source/pineapple_rl_lab/pineapple_rl_lab/assets/data/Robots/csl/pineapple/urdf/pineapple.urdf (robot description, URDF)
Before this commit: robot pineapple, 9 links, 8 joints
Joints:
- joint L_hip_joint: axis -1 0 0 -> 1 0 0
- joint R_hip_joint: axis -1 0 0 -> 1 0 0

Commit message: Update v1 urdf

File: source/pineapple_rl_lab/pineapple_rl_lab/assets/data/Robots/csl/pineapple/urdf/pineapple.urdf (robot description, URDF)
Before this commit: robot pineapple, 9 links, 8 joints
Links:
- removed link L_thgih
- added link L_thigh, mass 0.98; collision mesh filename=../meshes/L_thigh_collision.STL; visual mesh filename=../meshes/L_thigh.STL
- added link cam, mass 0.3; visual mesh filename=../meshes/cam.STL
Joints:
- added joint cam_joint: type fixed, parent base_link, child cam, origin xyz=0.136663127592924 0 0.125539913353642 rpy=0 0.698131700797732 0, axis 0 0 0
- joint L_calf_joint: parent L_thgih -> L_thigh
- joint L_hip_joint: limit lower=-0.52358 upper=0.52358 effort=23.7 velocity=30.1 -> lower=-0.52358 upper=0.17444 effort=23.7 velocity=30.1
- joint L_thigh_joint: child L_thgih -> L_thigh
- joint L_wheel_joint: limit lower=-999999 upper=999999 effort=3.69 velocity=60 -> effort=3.69 velocity=60.0
- joint R_hip_joint: limit lower=-0.52358 upper=0.52358 effort=23.7 velocity=30.1 -> lower=-0.17444 upper=0.52358 effort=23.7 velocity=30.1
- joint R_wheel_joint: limit lower=-999999 upper=999999 effort=3.69 velocity=60 -> effort=3.69 velocity=60.0

Commit message: Update urdf files

File: source/pineapple_rl_lab/pineapple_rl_lab/assets/data/Robots/csl/pineapple/urdf/pineapple.urdf (robot description, URDF)
Before this commit: robot pineapple_v1, 10 links, 9 joints
Links:
- removed link cam
- added link battery, mass 0.64; visual mesh filename=package://pineapple v1.1/meshes/battery.STL
- link L_calf: geometry collision box size=0.048 0.0236 0.093; visual mesh filename=package://pineapple v1.1/meshes/L_calf.STL
- link L_hip: geometry visual mesh filename=package://pineapple v1.1/meshes/L_hip.STL
- link L_thigh: mass 0.98 -> 0.911; geometry collision box size=0.055 0.019 0.12; collision cylinder length=0.035 radius=0.0515
- link L_wheel: mass 0.3 -> 0.35; geometry collision cylinder length=0.023 radius=0.07; visual mesh filename=package://pineapple v1.1/meshes/L_wheel.STL
- link R_calf: geometry collision box size=0.048 0.0236 0.093; visual mesh filename=package://pineapple v1.1/meshes/R_calf.STL
- link R_hip: geometry visual mesh filename=package://pineapple v1.1/meshes/R_hip.STL
- link R_thigh: mass 0.98 -> 0.911; geometry collision box size=0.055 0.019 0.12; collision cylinder length=0.035 radius=0.0515
- link R_wheel: mass 0.3 -> 0.35; geometry collision cylinder length=0.023 radius=0.07; visual mesh filename=package://pineapple v1.1/meshes/R_wheel.STL
- link base_link: mass 3.63 -> 2.99; geometry collision box size=0.05 0.05 0.1; collision box size=0.05 0.05 0.1
Joints:
- removed joint cam_joint
- added joint battery_fix: type fixed, parent base_link, child battery, origin xyz=0 0 0 rpy=0 0 0, axis 0 0 0
- joint L_calf_joint: origin xyz=0 0.04135 -0.165 rpy=0 0 0 -> xyz=0 0.0383 -0.165 rpy=0 0 0
- joint L_hip_joint: origin xyz=0 0.061689 0.066 rpy=0 0 0 -> xyz=0.047159 0.06125 0.066001 rpy=0 0 0
- joint L_thigh_joint: origin xyz=0 0.027596 0 rpy=0 0 0 -> xyz=-0.05675 0.01995 0 rpy=0 0 0
- joint L_wheel_joint: limit effort=3.69 velocity=60.0 -> effort=3.69 velocity=60; origin xyz=0 0.024414 -0.165 rpy=0 0 0 -> xyz=0 0.02705 -0.165 rpy=0 0 0; type revolute -> continuous
- joint R_calf_joint: origin xyz=0 -0.04135 -0.165 rpy=0 0 0 -> xyz=0 -0.0383 -0.165 rpy=0 0 0
- joint R_hip_joint: origin xyz=0 -0.061689 0.066 rpy=0 0 0 -> xyz=0.047159 -0.06125 0.066001 rpy=0 0 0
- joint R_thigh_joint: origin xyz=0 -0.027596 0 rpy=0 0 0 -> xyz=-0.05675 -0.01995 0 rpy=0 0 0
- joint R_wheel_joint: limit effort=3.69 velocity=60.0 -> effort=3.69 velocity=60; origin xyz=0 -0.024414 -0.165 rpy=0 0 0 -> xyz=0 -0.02705 -0.165 rpy=0 0 0; type revolute -> continuous

File: source/pineapple_rl_lab/pineapple_rl_lab/assets/data/Robots/csl/pineapple_v2/urdf/pineappleV2.urdf (robot description, URDF)
Before this commit: robot pineapple_v2, 18 links, 17 joints
Links:
- link L_calf: geometry collision box size=0.052 0.021 0.122; collision cylinder length=0.021 radius=0.026
- link L_hip: geometry visual mesh filename=../meshes/L_hip.STL
- link L_thigh: geometry collision box size=0.056 0.028 0.11; collision cylinder length=0.028 radius=0.028
- link L_wheel: geometry collision cylinder length=0.023 radius=0.077; visual mesh filename=../meshes/L_wheel.STL
- link R_calf: geometry collision box size=0.052 0.021 0.122; collision cylinder length=0.021 radius=0.026
- link R_hip: geometry visual mesh filename=../meshes/R_hip.STL
- link R_thigh: geometry collision box size=0.056 0.028 0.11; collision cylinder length=0.028 radius=0.028
- link R_wheel: geometry collision cylinder length=0.023 radius=0.077; visual mesh filename=../meshes/R_wheel.STL
- link arm_base: geometry visual mesh filename=../meshes/arm_base.STL
- link base_link: geometry collision box size=0.31 0.15 0.13; visual mesh filename=../meshes/base_link.STL
- link battery: geometry visual mesh filename=../meshes/battery.STL
- link camera: geometry visual mesh filename=../meshes/camera.STL
- link hip_motor_L: geometry visual mesh filename=../meshes/hip_motor_L.STL
- link hip_motor_R: geometry visual mesh filename=../meshes/hip_motor_R.STL
- link knee_motor_L: geometry visual mesh filename=../meshes/knee_motor_L.STL
- link knee_motor_R: geometry visual mesh filename=../meshes/knee_motor_R.STL
- link wheel_motor_L: geometry visual mesh filename=../meshes/wheel_motor_L.STL
- link wheel_motor_R: geometry visual mesh filename=../meshes/wheel_motor_R.STL

Commit message: Update sipo with right contact kinematics and non-holonomic constraint

File: source/pineapple_rl_lab/pineapple_rl_lab/assets/data/Robots/csl/pineapple/urdf/pineapple.urdf (robot description, URDF)
Before this commit: robot pineapple v1.1, 10 links, 9 joints
Links:
- link L_calf: geometry collision box size=0.048 0.0236 0.093; visual mesh filename=package://pineapple_v1/meshes/L_calf.STL
- link L_hip: geometry visual mesh filename=package://pineapple_v1/meshes/L_hip.STL
- link L_thigh: geometry collision box size=0.055 0.019 0.12; collision cylinder length=0.035 radius=0.0515
- link L_wheel: geometry collision cylinder length=0.023 radius=0.07; visual mesh filename=package://pineapple_v1/meshes/L_wheel.STL
- link R_calf: geometry collision box size=0.048 0.0236 0.093; visual mesh filename=package://pineapple_v1/meshes/R_calf.STL
- link R_hip: geometry visual mesh filename=package://pineapple_v1/meshes/R_hip.STL
- link R_thigh: geometry collision box size=0.055 0.019 0.12; collision cylinder length=0.035 radius=0.0515
- link R_wheel: geometry collision cylinder length=0.023 radius=0.07; visual mesh filename=package://pineapple_v1/meshes/R_wheel.STL
- link base_link: geometry collision box size=0.05 0.05 0.1; collision box size=0.05 0.05 0.1
- link battery: geometry visual mesh filename=package://pineapple_v1/meshes/battery.STL
Joints:
- joint L_wheel_joint: type continuous -> revolute
- joint R_wheel_joint: type continuous -> revolute
